File: PCB/ShutterController.sch (KiCad schematic (older format))
At the start: 27 parts, among them J1 Screw_Terminal_01x03, J2 Screw_Terminal_01x02, Q1 TS13003, Q2 TS13003, Q3 TS13003, Q4 TS13003, Q5 TS13003, Q6 TS13003, Q7 TS13003, U1 LM7805_TO220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

Commit message: Update
Parts:
- removed D1, D2, D3, D4: D, Diodes_THT:D_A-405_P10.16mm_Horizontal, symbol D
- removed Q5, Q6, Q7: TS13003, TO_SOT_Packages_THT:TO-92_Inline_Wide, symbol 2SC1815
- added D1, D2, D3, D4, D5: LED, LEDs:LED_D5.0mm, symbol LED
- added Q1, Q2, Q3, Q8, Q9: BC547, TO_SOT_Packages_THT:TO-92_Inline_Wide, symbol 2N2219
- added R10, R9: 100K, Resistors_THT:R_Axial_DIN0207_L6.3mm_D2.5mm_P10.16mm_Horizontal, symbol R
- added R14, R15, R16, R17, R18: 100, Resistors_THT:R_Axial_DIN0207_L6.3mm_D2.5mm_P10.16mm_Horizontal, symbol R
- added R7, R8: 47, Resistors_THT:R_Axial_DIN0207_L6.3mm_D2.5mm_P10.16mm_Horizontal, symbol R
- added RV1, RV3: 1K, Potentiometers:Potentiometer_Trimmer_Piher_PT-10v5_Horizontal_Px5.0mm_Py5.0mm, symbol POT_TRIM
- added RV2: 5K, Potentiometers:Potentiometer_Trimmer_Piher_PT-10v5_Horizontal_Px5.0mm_Py5.0mm, symbol POT_TRIM
- C1, C2: footprint Capacitors_THT:CP_Radial_D10.0mm_P2.50mm -> Capacitors_THT:CP_Radial_D10.0mm_P5.00mm
- Q4: renamed from Q1; value TS13003 -> BD437; footprint TO_SOT_Packages_THT:TO-92_Inline_Wide -> TO_SOT_Packages_THT:TO-220-3_Vertical
- R1, R2: value 100 -> 100K; footprint Resistors_THT:R_Axial_DIN0204_L3.6mm_D1.6mm_P7.62mm_Horizontal -> Resistors_THT:R_Axial_DIN0207_L6.3mm_D2.5mm_P10.16mm_Horizontal
- R11: renamed from R9; value 1K -> 1.5K; footprint Resistors_THT:R_Axial_DIN0204_L3.6mm_D1.6mm_P7.62mm_Horizontal -> Resistors_THT:R_Axial_DIN0207_L6.3mm_D2.5mm_P10.16mm_Horizontal
- R12: renamed from R8; footprint Resistors_THT:R_Axial_DIN0204_L3.6mm_D1.6mm_P7.62mm_Horizontal -> Resistors_THT:R_Axial_DIN0207_L6.3mm_D2.5mm_P10.16mm_Horizontal
- R13: renamed from R7; footprint Resistors_THT:R_Axial_DIN0204_L3.6mm_D1.6mm_P7.62mm_Horizontal -> Resistors_THT:R_Axial_DIN0207_L6.3mm_D2.5mm_P10.16mm_Horizontal
- R3: value 1K -> 100K; footprint Resistors_THT:R_Axial_DIN0204_L3.6mm_D1.6mm_P7.62mm_Horizontal -> Resistors_THT:R_Axial_DIN0207_L6.3mm_D2.5mm_P10.16mm_Horizontal
- R4: value 100 -> 47; footprint Resistors_THT:R_Axial_DIN0204_L3.6mm_D1.6mm_P7.62mm_Horizontal -> Resistors_THT:R_Axial_DIN0207_L6.3mm_D2.5mm_P10.16mm_Horizontal
- R5: value 810 -> 47; footprint Resistors_THT:R_Axial_DIN0204_L3.6mm_D1.6mm_P7.62mm_Horizontal -> Resistors_THT:R_Axial_DIN0207_L6.3mm_D2.5mm_P10.16mm_Horizontal
- R6: value 120 -> 47; footprint Resistors_THT:R_Axial_DIN0204_L3.6mm_D1.6mm_P7.62mm_Horizontal -> Resistors_THT:R_Axial_DIN0207_L6.3mm_D2.5mm_P10.16mm_Horizontal
- renumbered Q2 to Q5, Q3 to Q6, Q4 to Q7
Connections:
- net CLOSE: now also D3.2 (A), Q9.2 (B)
- net GND: now also R1.2, R2.2, R3.2, U2.15 (CLKOUT/OSC2/RA6), R10.1, R14.1, R15.1, R16.1, R17.1, R18.1, R9.1
- net HOLD: now also D2.2 (A), Q2.2 (B)
- net OPEN: now also D1.2 (A), Q1.2 (B)
- net LOWER: now reaches U2.11 (RB5)
- net LOWER: now also D4.2 (A), Q3.2 (B)
- net RAISE: now reaches U2.12 (RB6/T1OSC0/T1CKI/PGC)
- net RAISE: now also D5.2 (A), Q8.2 (B)
- net at R13.2: now also U2.6 (RB0/INT); no longer U2.4 (~MCLR~/Vpp/RA5)
- net at Q6.3 (B): now also RV3.1, RV3.2; no longer R4.2
- net at Q5.3 (B): now also R6.1; no longer R3.1
- net at R5.1: now also RV2.3
- net 12V: now reaches C1.1, J1.1 (Pin_1), U1.1 (VI)
- net 12V: now also Q4.2 (C), Q6.2 (C)
- net M_CLOSE: no longer names the net of R4.1
- net M_CLOSE: now also RV1.3; no longer R3.2
- net VCC renamed VDD
- net VDD: now also U2.4 (~MCLR~/Vpp/RA5), Q1.3 (C), Q2.3 (C), Q3.3 (C), Q8.3 (C), Q9.3 (C); no longer Q4.2 (C), Q6.2 (C)
- new net: Q4.3 (B), RV1.1, RV1.2, RV2.1, RV2.2
- new net: Q7.3 (B), R7.2
- new net: Q3.1 (E), R3.1, R6.2
- new net: Q9.1 (E), R10.2, R8.2
- new net: Q1.1 (E), R1.1, R4.2
- new net: Q2.1 (E), R2.1, R5.2
- new net: Q8.1 (E), R7.1, R9.2
- new net: R8.1, RV3.3
- new net: D1.1 (K), R14.2
- new net: D2.1 (K), R15.2
- new net: D3.1 (K), R16.2
- new net: D4.1 (K), R17.2
- new net: D5.1 (K), R18.2
- no-connect marks 12 -> 8
Other:
- moved on the sheet: J2, Q4, Q5, Q6, Q7, R11, R12, R13, U2
